File: hw/sch_pcb/USBSDREADER01.kicad_pcb (KiCad board)
At the start: 2 copper layers, 70.6 x 50.3 mm, 47 parts, among them IC1 MAX14502AETL+, J1 3.3V, J10 HEADER_1x02, J11 HEADER_1x02, J2 USB_B, J3 USB_A, J4 VBUS, J5 HEADER_2x07_PARALLEL, J6 HEADER_2x05_PARALLEL, J7 HEADER_2x04_PARALLEL, J8 HEADER_1x02, J9 SD_Card-FPS009-4200-0, M1 HOLE M3, M2 HOLE M3, M3 HOLE, M4 HOLE, U1 TS5A4594

Commit message: WIP
Parts:
- added Q1: NPN, Package_TO_SOT_SMD:SOT-23-3, B.Cu at (162.8, 118.0)
- added Q2: NPN, Package_TO_SOT_SMD:SOT-23-3, B.Cu at (159.3, 118.0)
- moved C1 80.7 mm to (171.5, 92.8), turned to 90 degrees
- moved D1 76.5 mm to (166.0, 92.5), turned to 90 degrees
- moved D3 60.6 mm to (172.1, 83.6), turned to 90 degrees
- moved D4 56.8 mm to (169.5, 83.6), turned to 90 degrees
- moved R12 51.2 mm to (157.3, 127.5)
- moved C2 48.1 mm to (169.5, 92.8), turned to 90 degrees
- moved C7 45.4 mm to (138.8, 98.7)
- moved R4 44.3 mm to (160.8, 127.5)
- moved R11 42.8 mm to (162.1, 114.1), turned to 90 degrees
- moved R5 42.1 mm to (164.3, 127.5)
- moved R13 35.3 mm to (148.3, 116.0)
- moved C8 30.9 mm to (151.1, 118.5)
- moved R10 29.3 mm to (159.8, 114.1), turned to 90 degrees
- moved R9 23.2 mm to (171.8, 88.0), turned to -90 degrees
- moved R6 22.4 mm to (155.0, 96.6)
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Connections:
- J7 pad 3: /mode -> /#RST
- J7 pad 4: /mode -> /#RST
- J7 pad 5: /i2c -> /mode
- J7 pad 6: /i2c -> /mode
- J7 pad 7: /#RST -> /i2c
- J7 pad 8: /#RST -> /i2c
- R10 pad 2: /#BERR -> /#BUSSY
- R11 pad 2: /#BUSSY -> /#BERR
- R12 pad 2: /mode -> /#RST
- R4 pad 2: /i2c -> /mode
- R5 pad 2: /#RST -> /i2c
Routing:
- net VCC: track 0.00 -> 52.9 mm, vias 0 -> 1
- net Net-(Q2-C): track 0.00 -> 52.0 mm, vias 0 -> 1
- net Net-(Q1-C): track 0.00 -> 46.4 mm, vias 0 -> 1
- net /SDA: track 0.00 -> 38.6 mm
- net /i2c: track 0.00 -> 35.6 mm, vias 0 -> 2
- net /SCL: track 0.00 -> 34.5 mm
- net /#RST: track 0.00 -> 31.5 mm
- net /mode: track 0.00 -> 29.3 mm
- net /#BERR: track 0.00 -> 17.9 mm
- net /i2c_addr: track 0.00 -> 17.6 mm, vias 0 -> 2
- net /#BUSSY: track 0.00 -> 16.0 mm
- net /USB_OUT_D+: track 16.8 -> 30.6 mm
- net /USB_OUT_D-: track 16.9 -> 30.6 mm
- net /SDP: track 0.00 -> 11.0 mm
- net /VIO: track 0.00 -> 6.54 mm
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- added copper zone on B.Cu, net GND
- added copper zone on F.Cu, net GND
