File: hw/sch_pcb/USBSDREADER01.kicad_sch (KiCad schematic)
At the start: 8 parts, among them J1 Umin ... Umax, M1 HOLE M3, M2 HOLE M3, M3 HOLE, M4 HOLE

Commit message: wip
Parts:
- added C10: 100nF, Capacitor_SMD:C_0805_2012Metric, symbol ISM02A-rescue:C_Small-Device-ISM02A-rescue
- added C3, C4, C5, C6, C7: C_Small, Capacitor_SMD:C_0805_2012Metric, symbol Device:C_Small
- added C8: 10uF, Capacitor_SMD:C_0805_2012Metric, symbol Device:C_Small
- added C9: 10uF, Capacitor_SMD:C_0805_2012Metric, symbol ISM02A-rescue:C_Small-Device-ISM02A-rescue
- added D2: BZV55C-5,6V, Diode_SMD:D_SMA, symbol ISM02A-rescue:D_ZENER-MLAB_D
- added D3, D4: LED, Mlab_D:LED_1206_mill, symbol Device:LED
- added FID1, FID2: Fiducial, Fiducial:Fiducial_0.5mm_Mask1mm, symbol Mechanical:Fiducial
- added IC1: MAX14502AETL+, Mlab_IO:QFN40P500X500X80-41N, symbol MLAB_IO:MAX14502AETL+
- added J10, J11: HEADER_1x02, Connector_PinHeader_2.54mm:PinHeader_1x02_P2.54mm_Vertical, symbol MLAB_HEADER:HEADER_1x02
- added J2: USB_B, Connector_USB:USB_B_Lumberg_2411_02_Horizontal, symbol Connector:USB_B
- added J3: USB_A, Connector_USB:USB_A_CONNFLY_DS1095-WNR0, symbol Connector:USB_A
- added J4: VBUS, Mlab_Pin_Headers:Straight_2x03, symbol header:HEADER_2x03_PARALLEL
- added J5: HEADER_2x07_PARALLEL, Connector_PinHeader_2.54mm:PinHeader_2x07_P2.54mm_Vertical, symbol MLAB_HEADER:HEADER_2x07_PARALLEL
- added J6: HEADER_2x05_PARALLEL, Connector_PinHeader_2.54mm:PinHeader_2x05_P2.54mm_Vertical, symbol MLAB_HEADER:HEADER_2x05_PARALLEL
- added J7: HEADER_2x04_PARALLEL, Connector_PinHeader_2.54mm:PinHeader_2x06_P2.54mm_Vertical, symbol MLAB_HEADER:HEADER_2x06_PARALLEL
- added J8: HEADER_1x02, Connector_PinHeader_2.54mm:PinHeader_1x03_P2.54mm_Vertical, symbol MLAB_HEADER:HEADER_1x03
- added J9: SD_Card-FPS009-4200-0, Mlab_CON:FPS009-4200-0, symbol MLAB_CONNECTORS:SD_Card-FPS009-4200-0
- added L1: 1uH, Inductor_SMD:L_1008_2520Metric, symbol Device:L_Small
- added Q1, Q2: NPN, symbol Simulation_SPICE:NPN
- added R1: 6.19k, Resistor_SMD:R_0805_2012Metric, symbol Device:R_Small
- added R10, R11, R6, R7, R8, R9: R_Small, Resistor_SMD:R_0805_2012Metric, symbol Device:R_Small
- added R12, R13, R2, R3, R4, R5: 10k, Resistor_SMD:R_0805_2012Metric, symbol Device:R_Small
- added U1: TS5A4594, Package_TO_SOT_SMD:SOT-23-5, symbol MLAB_IO:TS5A4594
- J1: value Umin ... Umax -> 3.3V
Connections:
- net GND: now also C10.2, C3.2, C4.2, C5.2, C6.2, C7.2, C8.2, C9.2, D2.2 (A), IC1.18 (GND_1), IC1.24 (GND_2), IC1.26 (GND_3), IC1.33 (CCRD_PRST), IC1.35 (N.C._1), IC1.36 (N.C._2), IC1.37 (GND_4), IC1.41 (GND_5), J2.4 (GND), J2.5 (Shield), J3.4 (GND), J3.5 (Shield), J4.1, J4.2, J4.5, J4.6, J6.1, J6.10, J6.2, J6.9, J8.1, J8.2, J8.3, J9.3 (VSS), J9.6 (VSS), Q1.3 (E), Q2.3 (E), R1.2, R3.2, R6.2, U1.3 (GND)
- net +5V renamed VCC
- net VCC: now also C4.1, D3.1 (K), D4.1 (K), IC1.39 (VCC), J6.5, J6.6, R12.1, R13.1, R4.1, R5.1, R7.1, U1.2 (NO), U1.5 (VCC)
- new net: D4.2 (A), R8.1
- new net: J7.11, J7.12, Q1.1 (C), R8.2
- new net: Q1.2 (B), R11.1
- new net: Q2.2 (B), R10.1
- new net: J7.10, J7.9, Q2.1 (C), R9.2
- new net: L1.2, U1.1 (COM)
- new net: D3.2 (A), R9.1
- new net: IC1.10 (CDAT1_3), J9.1 (CD/DAT3)
- new net: IC1.13 (CDAT1_0), J9.7 (DAT0)
- new net: IC1.12 (CDAT1_1), J9.8 (DAT1)
- new net: IC1.11 (CDAT1_2), J9.9 (DAT2)
- new net #BERR: IC1.6 (~{BERR}/INT), R10.2
- new net #BUSSY: IC1.7 (~{BUSY}), R11.2
- new net #RST: IC1.9 (~{RST}), J7.7, J7.8, R5.2
- new net CCLK: IC1.32 (CCLK1), J9.5 (CLK)
- new net CCMD: IC1.34 (CCMD1), J9.2 (CMD)
- new net CLDO: C5.1, IC1.38 (CLDO)
- new net CLK: IC1.29 (HCLK1), J5.13, J5.14
- new net CMD: IC1.31 (HCMD1), J5.11, J5.12
- new net DAT0: IC1.17 (HDAT1_0), J5.7, J5.8
- new net DAT1: IC1.16 (HDAT1_1), J5.5, J5.6
- new net DAT2: IC1.15 (HDAT1_2), J5.3, J5.4
- new net DAT3: IC1.14 (HDAT1_3), J5.1, J5.2
- new net KVBUS: IC1.28 (KVBUS), R2.2, R3.1
- new net PRST: IC1.30 (HCRD_PRST), J5.10, J5.9
- new net RREF: IC1.27 (RREF), R1.1
- new net SCL: IC1.2 (SCL), J6.7, J6.8
- new net SDA: IC1.3 (SDA), J6.3, J6.4
- new net SDP: J7.1, J7.2, R13.2, U1.4 (IN)
- new net USB_IN_D+: IC1.22 (CD+), J10.2, J2.3 (D+)
- new net USB_IN_D-: IC1.21 (CD-), J10.1, J2.2 (D-)
- new net USB_OUT_D+: IC1.20 (HD+), J11.1, J3.3 (D+)
- new net USB_OUT_D-: IC1.19 (HD-), J11.2, J3.2 (D-)
- new net VBUS: C10.1, C9.1, D2.1 (K), J2.1 (VBUS), J3.1 (VBUS), J4.3, J4.4, R2.1
- new net VIO: C6.1, IC1.5 (VIO)
- new net VSD: C3.1, C8.1, IC1.40 (VSD), J9.4 (VDD), L1.1
- new net VTM: C7.1, IC1.23 (VTM)
- new net i2c: IC1.1 (I2C_SEL), J7.5, J7.6, R4.2
- new net i2c_addr: IC1.4 (ADD), R6.1, R7.2
- new net mode: IC1.8 (MODE), J7.3, J7.4, R12.2
- no-connect marks 0 -> 1
Other:
- note removed: "Adjust power voltage range and symbol"
- note removed: "Delete if unused."
- note removed: "Generally a load module has mounting holes connected to the ground."
- note removed: "Power source modules has mountig holes floating to avoid ground loops."
- note removed: "check if the mounting holles should be connected to ground or not."
