File: hw/sch_pcb/USBSDREADER01.kicad_sch (KiCad schematic)
At the start: 49 parts, among them IC1 MAX14502AETL+, J1 3.3V, J10 HEADER_1x02, J11 HEADER_1x02, J2 USB_B, J3 USB_A, J4 VBUS, J5 HEADER_2x07_PARALLEL, J6 HEADER_2x05_PARALLEL, J7 HEADER_2x04_PARALLEL, J8 HEADER_1x02, J9 SD_Card-FPS009-4200-0, M1 HOLE M3, M2 HOLE M3, M3 HOLE, M4 HOLE, Q1 NPN, Q2 NPN, U1 TS5A4594

Commit message: WIP
Parts:
- Q1, Q2: footprint (none) -> Package_TO_SOT_SMD:SOT-23-3
Connections:
- net #BERR: now also R11.2; no longer R10.2
- net #BUSSY: now also R10.2; no longer R11.2
- net #RST: now also J7.3, J7.4, R12.2; no longer J7.7, J7.8, R5.2
- net i2c: now also J7.7, J7.8, R5.2; no longer J7.5, J7.6, R4.2
- net mode: now also J7.5, J7.6, R4.2; no longer J7.3, J7.4, R12.2
Changed lines of the file:
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@@
     (effects (font (size 1.524 1.524)) (justify left bottom))
   )
-  (label "#BERR" (at 204.47 104.14 180) (fields_autoplaced)
+  (label "#BERR" (at 204.47 119.38 180) (fields_autoplaced)
     (effects (font (size 1.524 1.524)) (justify right bottom))
   )
@@
     (effects (font (size 1.524 1.524)) (justify right bottom))
   )
-  (label "i2c" (at 233.68 106.68 180) (fields_autoplaced)
+  (label "i2c" (at 233.68 109.22 180) (fields_autoplaced)
     (effects (font (size 1.524 1.524)) (justify right bottom))
   )
@@
     (effects (font (size 1.524 1.524)) (justify right bottom))
   )
-  (label "mode" (at 233.68 104.14 180) (fields_autoplaced)
+  (label "mode" (at 233.68 106.68 180) (fields_autoplaced)
     (effects (font (size 1.524 1.524)) (justify right bottom))
   )
@@
     (effects (font (size 1.524 1.524)) (justify right bottom))
   )
-  (label "#BUSSY" (at 204.47 119.38 180) (fields_autoplaced)
-    (effects (font (size 1.524 1.524)) (justify right bottom))
-  )
-  (label "#RST" (at 233.68 109.22 180) (fields_autoplaced)
+  (label "#BUSSY" (at 204.47 104.14 180) (fields_autoplaced)
+    (effects (font (size 1.524 1.524)) (justify right bottom))
+  )
+  (label "#RST" (at 233.68 104.14 180) (fields_autoplaced)
     (effects (font (size 1.524 1.524)) (justify right bottom))
   )
@@
   (symbol (lib_id "Mechanical:Fiducial") (at 266.7 62.23 0) (unit 1)
     (in_bom yes) (on_board yes) (dnp no) (fields_autoplaced)
-    (property "Reference" "FID2" (at 269.24 60.96 0)
+    (property "Reference" "FID2" (at 269.24 62.23 0)
       (effects (font (size 1.27 1.27)) (justify left))
     )
     (property "Value" "Fiducial" (at 269.24 63.5 0)
-      (effects (font (size 1.27 1.27)) (justify left))
+      (effects (font (size 1.27 1.27)) (justify left) hide)
     )
     (property "Footprint" "Fiducial:Fiducial_0.5mm_Mask1mm" (at 266.7 62.23 0)
@@
       (effects (font (size 1.27 1.27)) (justify left))
     )
-    (property "Footprint" "" (at 278.13 119.38 0)
+    (property "Footprint" "Package_TO_SOT_SMD:SOT-23-3" (at 278.13 119.38 0)
       (effects (font (size 1.27 1.27)) hide)
     )
@@
   (symbol (lib_id "Mechanical:Fiducial") (at 255.27 62.23 0) (unit 1)
     (in_bom yes) (on_board yes) (dnp no) (fields_autoplaced)
-    (property "Reference" "FID1" (at 257.81 60.96 0)
+    (property "Reference" "FID1" (at 257.81 62.23 0)
       (effects (font (size 1.27 1.27)) (justify left))
     )
     (property "Value" "Fiducial" (at 257.81 63.5 0)
-      (effects (font (size 1.27 1.27)) (justify left))
+      (effects (font (size 1.27 1.27)) (justify left) hide)
     )
     (property "Footprint" "Fiducial:Fiducial_0.5mm_Mask1mm" (at 255.27 62.23 0)
@@
       (effects (font (size 1.27 1.27)) (justify left))
     )
-    (property "Footprint" "" (at 278.13 104.14 0)
-      (effects (font (size 1.27 1.27)) hide)
-    )
+    (property "Footprint" "Package_TO_SOT_SMD:SOT-23-3" (at 278.13 104.14 0)
+      (effects (font (size 1.27 1.27)) hide)
+    )

Commit message: Update documentation.
Other:
- title: NAME -> USBSDREADER01A
Changed lines of the file:
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@@
   (paper "A4")
   (title_block
-    (title "NAME")
+    (title "USBSDREADER01A")
     (date "%d. %m. %Y")
     (rev "REV")
     (company "Mlab www.mlab.cz")
-    (comment 1 "Short description \\nTwo lines are maximum")
+    (comment 1 "USB to SD Card Reader\\nsupports USB 2.0 and SDHC cards.")
     (comment 2 "nickname <email@example.com>")
   )
